File: board/Retro_Programmer-v0.1.brd (EAGLE design)
At the start: 45 x 45 mm, 48 parts, among them IC1 74LVC125A, K1 61301511821, K2 61301511821, P1 POWERSUPPLY_DC21MMX, Q1 BC857CSMD, Q2 BC847, SW1 SPUSH, SW2 SPUSH, SW3 SPUSH, SW4 SLIDE_WAY4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

Commit message: More bla bla bla
Parts:
- C2: value 100n -> 100nF
- C5: value 10uF -> 100nF
Changed lines of the file:
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@@
 <layer number="19" name="Unrouted" color="6" fill="1" visible="yes" active="yes"/>
 <layer number="20" name="Dimension" color="15" fill="1" visible="yes" active="yes"/>
-<layer number="21" name="tPlace" color="7" fill="1" visible="no" active="yes"/>
+<layer number="21" name="tPlace" color="7" fill="1" visible="yes" active="yes"/>
 <layer number="22" name="bPlace" color="7" fill="1" visible="yes" active="yes"/>
-<layer number="23" name="tOrigins" color="15" fill="1" visible="no" active="yes"/>
+<layer number="23" name="tOrigins" color="15" fill="1" visible="yes" active="yes"/>
 <layer number="24" name="bOrigins" color="15" fill="1" visible="yes" active="yes"/>
-<layer number="25" name="tNames" color="7" fill="1" visible="no" active="yes"/>
+<layer number="25" name="tNames" color="7" fill="1" visible="yes" active="yes"/>
 <layer number="26" name="bNames" color="7" fill="1" visible="yes" active="yes"/>
 <layer number="27" name="tValues" color="7" fill="1" visible="no" active="yes"/>
@@
 <attribute name="VALUE" x="34.2884" y="40.3554" size="1.27" layer="28" rot="MR90"/>
 </element>
-<element name="C2" library="rcl" package="C1206" value="100n" x="40.0204" y="41.6508" smashed="yes" rot="MR90">
+<element name="C2" library="rcl" package="C1206" value="100nF" x="40.0204" y="41.6508" smashed="yes" rot="MR90">
 <attribute name="NAME" x="41.6714" y="38.8568" size="0.8128" layer="26" rot="MR90"/>
 <attribute name="VALUE" x="37.4804" y="40.3808" size="1.27" layer="28" rot="MR90"/>
@@
 <attribute name="VALUE" x="26.27" y="5.94" size="1.27" layer="27" rot="R180"/>
 </element>
-<element name="C5" library="rcl" package="C1206" value="10uF" x="37.9158" y="9.392" smashed="yes">
+<element name="C5" library="rcl" package="C1206" value="100nF" x="37.9158" y="9.392" smashed="yes">
 <attribute name="NAME" x="40.6844" y="7.995" size="0.6096" layer="25"/>
 <attribute name="VALUE" x="36.6458" y="6.852" size="1.27" layer="27"/>
