File: board/Retro_Programmer-v0.2.sch (EAGLE design)
At the start: 48 parts, among them IC1 74LVC125A, K1 61301511821, K2 61301511821, P1 POWERSUPPLY_DC21MMX, Q1 BC857CSMD, Q2 BC847, SW1 SPUSH, SW2 SPUSH, SW3 SPUSH, SW4 SLIDE_WAY4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

Commit message: Board: Fixed ICSP+TID label, and other labels
Parts:
- renumbered ICSP+TD to ICSP+TID
Changed lines of the file:
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@@
 <setting verticaltext="up"/>
 </settings>
-<grid distance="0.01" unitdist="inch" unit="inch" style="lines" multiple="1" display="no" altdistance="0.01" altunitdist="inch" altunit="inch"/>
+<grid distance="0.1" unitdist="inch" unit="inch" style="lines" multiple="1" display="no" altdistance="0.01" altunitdist="inch" altunit="inch"/>
 <layers>
 <layer number="1" name="Top" color="4" fill="1" visible="no" active="no"/>
@@
 <part name="R6" library="rcl" deviceset="R-US_" device="R1206" value="22K"/>
 <part name="GND6" library="supply1" deviceset="GND" device=""/>
-<part name="ICSP+TD" library="Wuerth_Elektronik_Board_to_Board" deviceset="61301021821" device=""/>
+<part name="ICSP+TID" library="Wuerth_Elektronik_Board_to_Board" deviceset="61301021821" device=""/>
 <part name="GND7" library="supply1" deviceset="GND" device=""/>
 <part name="C2" library="rcl" deviceset="C-EU" device="C1206" value="100nF"/>
@@
 <instance part="R6" gate="G$1" x="40.64" y="43.18" rot="R90"/>
 <instance part="GND6" gate="1" x="40.64" y="19.05"/>
-<instance part="ICSP+TD" gate="G$1" x="205.74" y="54.61"/>
+<instance part="ICSP+TID" gate="G$1" x="205.74" y="54.61"/>
 <instance part="GND7" gate="1" x="156.21" y="68.58"/>
 <instance part="C2" gate="G$1" x="152.4" y="153.67"/>
@@
 <pinref part="R15" gate="G$1" pin="1"/>
 <wire x1="215.9" y1="60.96" x2="215.9" y2="59.69" width="0.1524" layer="91"/>
-<pinref part="ICSP+TD" gate="G$1" pin="1"/>
+<pinref part="ICSP+TID" gate="G$1" pin="1"/>
 <wire x1="213.36" y1="59.69" x2="215.9" y2="59.69" width="0.1524" layer="91"/>
 <wire x1="215.9" y1="59.69" x2="219.71" y2="59.69" width="0.1524" layer="91"/>
@@
 <segment>
 <pinref part="R14" gate="G$1" pin="1"/>
-<pinref part="ICSP+TD" gate="G$1" pin="10"/>
+<pinref part="ICSP+TID" gate="G$1" pin="10"/>
 <wire x1="198.12" y1="59.69" x2="191.77" y2="59.69" width="0.1524" layer="91"/>
 <wire x1="191.77" y1="59.69" x2="191.77" y2="62.23" width="0.1524" layer="91"/>
@@
 </segment>
 <segment>
-<pinref part="ICSP+TD" gate="G$1" pin="2"/>
+<pinref part="ICSP+TID" gate="G$1" pin="2"/>
 <wire x1="213.36" y1="57.15" x2="228.6" y2="57.15" width="0.1524" layer="91"/>
 <pinref part="R16" gate="G$1" pin="1"/>
@@
 </segment>
 <segment>
-<pinref part="ICSP+TD" gate="G$1" pin="4"/>
+<pinref part="ICSP+TID" gate="G$1" pin="4"/>
 <wire x1="213.36" y1="52.07" x2="219.71" y2="52.07" width="0.1524" layer="91"/>
 <label x="219.71" y="52.07" size="1.27" layer="95" xref="yes"/>
@@
 </segment>
 <segment>
-<pinref part="ICSP+TD" gate="G$1" pin="6"/>
+<pinref part="ICSP+TID" gate="G$1" pin="6"/>
 <wire x1="198.12" y1="49.53" x2="191.77" y2="49.53" width="0.1524" layer="91"/>
 <label x="191.77" y="49.53" size="1.27" layer="95" rot="R180" xref="yes"/>
@@
 </segment>
 <segment>
-<pinref part="ICSP+TD" gate="G$1" pin="7"/>
+<pinref part="ICSP+TID" gate="G$1" pin="7"/>
 <wire x1="198.12" y1="52.07" x2="195.58" y2="52.07" width="0.1524" layer="91"/>
 <label x="195.58" y="52.07" size="1.27" layer="95" rot="R180" xref="yes"/>
@@
 </segment>
 <segment>
-<pinref part="ICSP+TD" gate="G$1" pin="8"/>
+<pinref part="ICSP+TID" gate="G$1" pin="8"/>
 <wire x1="198.12" y1="54.61" x2="191.77" y2="54.61" width="0.1524" layer="91"/>
 <label x="191.77" y="54.61" size="1.27" layer="95" rot="R180" xref="yes"/>
@@
 </segment>
 <segment>
-<pinref part="ICSP+TD" gate="G$1" pin="3"/>
+<pinref part="ICSP+TID" gate="G$1" pin="3"/>
 <wire x1="213.36" y1="54.61" x2="232.41" y2="54.61" width="0.1524" layer="91"/>
 <wire x1="232.41" y1="54.61" x2="232.41" y2="52.07" width="0.1524" layer="91"/>
@@
 <net name="D3ENB" class="0">
 <segment>
-<pinref part="ICSP+TD" gate="G$1" pin="5"/>
+<pinref part="ICSP+TID" gate="G$1" pin="5"/>
 <wire x1="213.36" y1="49.53" x2="218.44" y2="49.53" width="0.1524" layer="91"/>
 <label x="218.44" y="45.72" size="1.27" layer="95" xref="yes"/>
